File: md2.kicad_sch (KiCad schematic)
At the start: 39 parts, among them IC1 TC74HC4066AP_F_, IC2 TC74HC4066AP_F_, IC3 TC74HC04AP, IC4 TB6643KQ, IC5 TB6643KQ, IC6 TB6643KQ, IC7 TB6643KQ, J1 Conn_01x03_Pin, J10 Conn_01x02_Pin, J11 Conn_01x01_Pin, J2 Conn_01x03_Pin, J3 Conn_01x03_Pin, J4 Conn_01x03_Pin, J5 XT30PW-M, J6 XT30PW-M, J7 XT30PW-M, J8 XT30PW-M, J9 Conn_01x02_Pin, SW1 SW_Push, SW2 SW_Push, SW3 SW_Push, SW4 SW_Push, SW5 SW_Push, SW6 SW_Push, SW7 SW_Push, SW8 SW_Push, SW9 SW_Push, U1 NJM7805FA

Commit message: Update
Parts:
- added C1, C3: 1u, Capacitor_THT:C_Disc_D6.0mm_W4.4mm_P5.00mm, symbol Device:C
- added C13, C14, C15, C16, C17, C18: 0.1u, Capacitor_THT:C_Disc_D6.0mm_W4.4mm_P5.00mm, symbol Device:C
- added D1: LED, LED_THT:LED_D3.0mm, symbol Device:LED
- added R10, R11, R2, R3, R4, R5, R6, R7, R8, R9: 10k, Resistor_THT:R_Axial_DIN0207_L6.3mm_D2.5mm_P10.16mm_Horizontal, symbol Device:R
- added R12: 1k, Resistor_THT:R_Axial_DIN0207_L6.3mm_D2.5mm_P10.16mm_Horizontal, symbol Device:R
- added U2: SeeeduinoXIAO, Seeeduino XIAO KICAD:Seeeduino XIAO-MOUDLE14P-2.54-21X17.8MM, symbol Seeeduino XIAO:SeeeduinoXIAO
- C4: value 10u -> 0.1u; footprint Capacitor_THT:CP_Radial_D5.0mm_P2.00mm -> Capacitor_THT:C_Disc_D6.0mm_W4.4mm_P5.00mm
- C8: value 220u -> 0.1u; footprint Capacitor_THT:CP_Radial_D8.0mm_P3.50mm -> Capacitor_THT:C_Disc_D6.0mm_W4.4mm_P5.00mm
Connections:
- net +5V: now also C1.1; no longer C4.1
- net CW/CCW-1: now also C15.1, R8.2, U2.2 (PA4_A1_D1)
- net CW/CCW-2: now also C16.1, R9.2, U2.4 (PA11_A3_D3)
- net CW/CCW-3: now also C17.1, R10.2, U2.6 (PA9_A5_D5_SCL)
- net CW/CCW-4: now also C18.1, R11.2, U2.10 (PA5_A9_D9_MISO)
- net GND: now also C1.2, C13.2, C14.2, C15.2, C16.2, C17.2, C18.2, C3.2, R10.1, R11.1, R12.1, R2.1, R3.1, R4.1, R5.1, R6.1, R7.1, R8.1, R9.1, U2.13 (GND)
- net PWM-1: now also C4.1, R2.2, U2.1 (PA02_A0_D0)
- net PWM-2: now also C8.1, R3.2, U2.3 (PA10_A2_D2)
- net PWM-3: now also C13.1, R4.2, U2.5 (PA8_A4_D4_SDA)
- net PWM-4: now also C14.1, R5.2, U2.11 (PA6_A10_D10_MOSI)
- net VDD: now also C3.1, D1.2 (A); no longer C8.1
- net at IC3.11 (5A): now also R7.2
- net at IC3.13 (6A): now also R6.2
- new net: D1.1 (K), R12.2
Other:
- moved on the sheet: C2, C5, C6, C7, IC1, IC2, IC3, J1, J10, J2, J3, J4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

Commit message: update
Parts:
- removed C10, C11, C12, C9: 0.1u, Capacitor_THT:C_Disc_D6.0mm_W4.4mm_P5.00mm, symbol Device:C
- removed J1, J2, J3, J4: Conn_01x03_Pin, Connector_PinHeader_2.54mm:PinHeader_1x03_P2.54mm_Vertical, symbol Connector:Conn_01x03_Pin
- removed J11: Conn_01x01_Pin, led:led_conn, symbol Connector:Conn_01x01_Pin
- removed R1: R, Resistor_THT:R_Axial_DIN0207_L6.3mm_D2.5mm_P10.16mm_Horizontal, symbol Device:R
- removed R10, R11, R2, R3, R4, R5, R8, R9: 10k, Resistor_THT:R_Axial_DIN0207_L6.3mm_D2.5mm_P10.16mm_Horizontal, symbol Device:R
- added J1: Conn_01x02_Pin, Connector_PinHeader_2.54mm:PinHeader_1x02_P2.54mm_Vertical, symbol Connector:Conn_01x02_Pin
- added J3: Conn_02x13_Odd_Even, Connector_PinSocket_1.27mm:PinSocket_2x13_P1.27mm_Vertical, symbol Connector_Generic:Conn_02x13_Odd_Even
- added JP1: SolderJumper_2_Open, Jumper:SolderJumper-2_P1.3mm_Open_TrianglePad1.0x1.5mm, symbol Jumper:SolderJumper_2_Open
- added JP2, JP6: SolderJumper_3_Open, Jumper:SolderJumper-3_P1.3mm_Open_Pad1.0x1.5mm, symbol Jumper:SolderJumper_3_Open
- added RN1, RN2: 4609M-101-103LF, 4609M-101-103LF:4609X, symbol 4609M-101-103LF:4609M-101-103LF
Connections:
- net +5V: now also J1.1 (Pin_1), JP1.2 (B)
- net CW/CCW-1: now also RN1.4; no longer C15.1
- net CW/CCW-2: now also RN1.8; no longer C16.1
- net CW/CCW-3: now also RN2.2; no longer C17.1
- net CW/CCW-4: now also RN2.5; no longer C18.1
- net GND: now also J3.24 (Pin_24), RN1.1, RN2.1
- net MD-1-1: now also C14.1, RN1.2
- net MD-1-2: now also C13.1, RN1.3
- net MD-2-1: now also C4.1, RN1.7
- net MD-2-2: now also C8.1, RN1.9
- net MD-3-1: now also C18.1, RN2.9
- net MD-3-2: now also C17.1, RN2.8
- net MD-4-1: now also C16.1, RN2.4
- net MD-4-2: now also C15.1, RN2.3
- net PWM-1: now also RN1.5; no longer C4.1
- net PWM-2: now also RN1.6; no longer C8.1
- net PWM-3: now also RN2.7; no longer C13.1
- net PWM-4: now also RN2.6; no longer C14.1
- net +3V3: now reaches U2.12 (3V3)
- net +3V3: now also J3.23 (Pin_23), J3.25 (Pin_25)
- net at U2.14 (5V): now also J1.2 (Pin_2), JP1.1 (A)
- net at U2.7 (PB08_A6_D6_TX): now also JP2.2 (C)
- net at U2.8 (PB09_A7_D7_RX): now also JP6.2 (C)
- net IM920-BUSY: now reaches U2.9 (PA7_A8_D8_SCK)
- net IM920-BUSY: now also J3.1 (Pin_1)
- new net IM920-RX: J3.6 (Pin_6), JP2.3 (B), JP6.3 (B)
- new net IM920-TX: J3.7 (Pin_7), JP2.1 (A), JP6.1 (A)

Commit message: update
Parts:
- removed C13, C14, C15, C16, C17, C18, C4, C8: 0.1u, Capacitor_THT:C_Disc_D6.0mm_W4.4mm_P5.00mm, symbol Device:C
- added D2: LED, LED_THT:LED_D3.0mm, symbol Device:LED
- added H1: 3557-15, 3557-15:355715, symbol 3557-15:3557-15
- added R1: 1k, Resistor_THT:R_Axial_DIN0207_L6.3mm_D2.5mm_P10.16mm_Horizontal, symbol Device:R
Connections:
- net CW/CCW-4: now also U2.9 (PA7_A8_D8_SCK); no longer U2.10 (PA5_A9_D9_MISO)
- net GND: now also R1.1; no longer J5.3, J5.4, J6.3, J6.4, J7.3, J7.4, J8.3, J8.4
- net IM920-BUSY: now also D2.2 (A); no longer U2.9 (PA7_A8_D8_SCK)
- net VDD: now also H1.3, H1.4; no longer SW9.2
- new net: H1.1, H1.2, SW9.2
- new net: D2.1 (K), R1.2
Other:
- moved on the sheet: J1, J3, JP1, JP2, JP6, U2

Commit message: update
Parts:
- removed D2: LED, LED_THT:LED_D3.0mm, symbol Device:LED
- removed R1: 1k, Resistor_THT:R_Axial_DIN0207_L6.3mm_D2.5mm_P10.16mm_Horizontal, symbol Device:R
- added D3, D4, D5, D6: D, Diode_THT:D_DO-41_SOD81_P10.16mm_Horizontal, symbol Device:D
Connections:
- net GND: now also D3.2 (A), D4.2 (A), D5.2 (A), D6.2 (A)
- net MD-1-2: now also IC1.3 (2O/I); no longer IC1.4 (2I/O)
- net MD-3-2: now also IC2.3 (2O/I); no longer IC2.4 (2I/O)
- net VDD: now also D3.1 (K), D4.1 (K), D5.1 (K), D6.1 (K)
- net r-CW/CCW-1: now also IC1.4 (2I/O); no longer IC1.3 (2O/I)
- net r-CW/CCW-3: now also IC2.4 (2I/O); no longer IC2.3 (2O/I)
- net IM920-BUSY: no longer names the net of J3.1 (Pin_1)
Other:
- moved on the sheet: C1, C2, IC4, IC5, IC6, IC7, J5, J6, J7, J8
